Commit message: new assets generated

File: urdf_output/iiwa7.urdf (robot description, URDF)
Before this commit: robot iiwa7, 1 links, 0 joints
Links:
- removed link world
- added link iiwa_link_0, mass 5; collision mesh filename=package://iiwa_description/meshes/iiwa7/collision/link_0.stl; visual mesh filename=package://iiwa_description/meshes/iiwa7/visual/link_0.stl
- added link iiwa_link_1, mass 3.4525; collision mesh filename=package://iiwa_description/meshes/iiwa7/collision/link_1.stl; visual mesh filename=package://iiwa_description/meshes/iiwa7/visual/link_1.stl
- added link iiwa_link_2, mass 3.4821; collision mesh filename=package://iiwa_description/meshes/iiwa7/collision/link_2.stl; visual mesh filename=package://iiwa_description/meshes/iiwa7/visual/link_2.stl
- added link iiwa_link_3, mass 4.05623; collision mesh filename=package://iiwa_description/meshes/iiwa7/collision/link_3.stl; visual mesh filename=package://iiwa_description/meshes/iiwa7/visual/link_3.stl
- added link iiwa_link_4, mass 3.4822; collision mesh filename=package://iiwa_description/meshes/iiwa7/collision/link_4.stl; visual mesh filename=package://iiwa_description/meshes/iiwa7/visual/link_4.stl
- added link iiwa_link_5, mass 2.1633; collision mesh filename=package://iiwa_description/meshes/iiwa7/collision/link_5.stl; visual mesh filename=package://iiwa_description/meshes/iiwa7/visual/link_5.stl
- added link iiwa_link_6, mass 2.3466; collision mesh filename=package://iiwa_description/meshes/iiwa7/collision/link_6.stl; visual mesh filename=package://iiwa_description/meshes/iiwa7/visual/link_6.stl
- added link iiwa_link_7, mass 3.129; collision mesh filename=package://iiwa_description/meshes/iiwa7/collision/link_7.stl; visual mesh filename=package://iiwa_description/meshes/iiwa7/visual/link_7.stl
- added link iiwa_link_ee
Joints:
- added joint iiwa_joint_1: type revolute, parent iiwa_link_0, child iiwa_link_1, origin xyz=0 0 0.15 rpy=0 0 0, axis 0 0 1, limit lower=-2.96706 upper=2.96706 effort=300 velocity=10
- added joint iiwa_joint_2: type revolute, parent iiwa_link_1, child iiwa_link_2, origin xyz=0 0 0.19 rpy=1.570796   0 3.1415926535897931, axis 0 0 1, limit lower=-2.094395 upper=2.094395 effort=300 velocity=10
- added joint iiwa_joint_3: type revolute, parent iiwa_link_2, child iiwa_link_3, origin xyz=0 0.21 0 rpy=1.570796 0 3.1415926535897931, axis 0 0 1, limit lower=-2.96706 upper=2.96706 effort=300 velocity=10
- added joint iiwa_joint_4: type revolute, parent iiwa_link_3, child iiwa_link_4, origin xyz=0 0 0.19 rpy=1.570796 0 0, axis 0 0 1, limit lower=-2.094395 upper=2.094395 effort=300 velocity=10
- added joint iiwa_joint_5: type revolute, parent iiwa_link_4, child iiwa_link_5, origin xyz=0 0.21 0 rpy=-1.570796 3.1415926535897931 0, axis 0 0 1, limit lower=-2.96706 upper=2.96706 effort=300 velocity=10
- added joint iiwa_joint_6: type revolute, parent iiwa_link_5, child iiwa_link_6, origin xyz=0 0.06070 0.19 rpy=1.570796 0 0, axis 0 0 1, limit lower=-2.094395 upper=2.094395 effort=300 velocity=10
- added joint iiwa_joint_7: type revolute, parent iiwa_link_6, child iiwa_link_7, origin xyz=0 0.081 0.06070 rpy=-1.570796 3.1415926535897931 0, axis 0 0 1, limit lower=-3.054326 upper=3.054326 effort=300 velocity=10
- added joint iiwa_joint_ee: type fixed, parent iiwa_link_7, child iiwa_link_ee, origin xyz=0 0 0.045 rpy=0 0 0
